File: MVME712M_P2_Adapter.kicad_pcb (KiCad board)
At the start: 4 copper layers, 100 x 80 mm, 13 parts, among them J1 Conn_01x05_Pin, J2 DIN41612_03x32_C_Split, J3 Conn_02x25_Odd_Even, P2 DIN41612_03x32_C_Split

Commit message: added RS232 text
Parts:
- removed G***: LOGO, LOGO
- D1: value 1N4148 -> 1N5819
- F1: value Fuse -> TRF250-120T-R2-B-0.5; footprint Fuse:Fuse_2512_6332Metric_Pad1.52x3.35mm_HandSolder -> Fuse:Fuse_Bourns_MF-RG500
- moved F1 2.90 mm to (114.0, 82.0)
Routing:
- net SEL: track 83.0 -> 85.2 mm
- net TERMPWR: track 58.8 -> 60.4 mm
- net REQ: track 77.2 -> 78.4 mm
- net TXD2: track 69.6 -> 70.7 mm
Other:
- board size 100 x 80 mm -> 100 x 78.7 mm
- board text added: "03.12.2025"
- board text added: "1"
- board text added: "MVME P2 Adapter Board"
- board text added: "Rev. 1 denis2342 parceval"
- board text added: "Serial 1 RS232 Levels"
- board text removed: "28.11.2025"
- board text removed: "P2 Adapter Module"
- board text removed: "Serial 1"

Commit message: added RS232 text on pcb
Other:
- board text added: "23.12.2025"
- board text removed: "03.12.2025"
Changed lines of the file:
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@@
 		)
 	)
-	(gr_text "03.12.2025"
+	(gr_text "23.12.2025"
 		(at 42 71.5 90)
 		(layer "F.SilkS")
